File: cpld_and_io.sch (KiCad schematic (older format))
At the start: 42 parts, among them J7 PMOD, J8 PMOD, SW1 SW_Push, SW2 SW_Push, U11 5M570ZT100I5N, U12 IS61LV5128AL-10TLI, X1 CB3LV-3I-50M0000

Commit message: Added logo, cpio vcc selection
Changed lines of the file:
@@
 Text GLabel 7370 3530 0    50   3State ~ 0
 D0_F
-Text GLabel 7370 4930 0    50   Input ~ 0
+Text GLabel 10570 2430 2    50   Input ~ 0
 ~BUSACK_F
-Text GLabel 7370 4830 0    50   Input ~ 0
+Text GLabel 10570 2530 2    50   Input ~ 0
 ~PAGE_F
-Text GLabel 7370 4430 0    50   Input ~ 0
+Text GLabel 10570 2930 2    50   Input ~ 0
 ~MREQ_F
-Text GLabel 7370 4530 0    50   Input ~ 0
+Text GLabel 10570 2830 2    50   Input ~ 0
 ~WR_F
-Text GLabel 7370 4630 0    50   Input ~ 0
+Text GLabel 10570 2730 2    50   Input ~ 0
 ~RD_F
-Text GLabel 7370 4730 0    50   Input ~ 0
+Text GLabel 10570 2630 2    50   Input ~ 0
 ~IORQ_F
-Text GLabel 7370 4330 0    50   Input ~ 0
+Text GLabel 10570 3030 2    50   Input ~ 0
 ~M1_F
 Text GLabel 7370 2430 0    50   Input ~ 0
@@
 Text GLabel 10570 1730 2    50   Output ~ 0
 ~RESET_F
-Text GLabel 10570 2830 2    50   Output ~ 0
+Text GLabel 6040 1990 2    50   Output ~ 0
 RX_A_F
 $Comp
@@
 Text GLabel 4350 6200 2    50   3State ~ 0
 GPIO_16
+Text GLabel 7370 5030 0    50   3State ~ 0
+D7_F
+Text GLabel 7370 4930 0    50   3State ~ 0
+D6_F
+Text GLabel 7370 4830 0    50   3State ~ 0
+D5_F
+Text GLabel 7370 4730 0    50   3State ~ 0
+D4_F
+Text GLabel 7370 4630 0    50   3State ~ 0
+D3_F
+Text GLabel 7370 4530 0    50   3State ~ 0
+D2_F
+Text GLabel 7370 4430 0    50   3State ~ 0
+D1_F
+Text GLabel 7370 4330 0    50   3State ~ 0
+D0_F
 $EndSCHEMATC

Commit message: larger maxv, additional clocks, reorganized sheets
Parts:
- removed C36, C37, C38, C39, C40, C41, C42, C43, C44, C45, C46, C47, C48, C49: 100nF, Capacitor_SMD:C_0603_1608Metric_Pad1.05x0.95mm_HandSolder, symbol Device:C
- removed D1, D2, D3, D4, D5, D6, D7, D8: Blue, LED_SMD:LED_0603_1608Metric_Pad1.05x0.95mm_HandSolder, symbol Device:LED_Small
- removed D10, D11, D12, D9: SP0504BAHT, Package_TO_SOT_SMD:SOT-23-5, symbol Power_Protection:SP0504BAHT
- removed J7, J8: PMOD, Connector_PinSocket_2.54mm:PinSocket_2x06_P2.54mm_Horizontal, symbol Connector_Generic:Conn_02x06_Top_Bottom
- removed R7, R8: 10K, Resistor_SMD:R_0603_1608Metric_Pad1.05x0.95mm_HandSolder, symbol Device:R_Small
- removed R9: 22R5, Resistor_SMD:R_0603_1608Metric_Pad1.05x0.95mm_HandSolder, symbol Device:R_Small
- removed RN4, RN5, RN6, RN7, RN8, RN9: 200R, Resistor_SMD:R_Array_Concave_4x0603, symbol Device:R_Pack04
- removed SW1, SW2: SW_Push, Button_Switch_SMD:SW_SPST_CK_RS282G05A3, symbol Switch:SW_Push
- removed U11: 5M570ZT100I5N, Package_QFP:TQFP-100_14x14mm_P0.5mm, symbol rc2014_max_v-rescue:5M570ZT100I5N
- removed X1: CB3LV-3I-50M0000, Oscillator:Oscillator_SMD_SeikoEpson_SG8002CA-4Pin_7.0x5.0mm_HandSoldering, symbol rc2014_max_v-rescue:CB3LV-3I-50M0000-Oscillator
- added RN10: 10K, Resistor_SMD:R_Array_Concave_4x0603, symbol Device:R_Pack04
- added U4: 5M1270ZT144C5N, Package_QFP:TQFP-144_20x20mm_P0.5mm, symbol CPLD_Altera:5M1270ZT144C5N
Connections:
- net labels added: D10_F, D11_F, D12_F, D13_F, D14_F, D15_F, D8_F, D9_F, GPIO_10_F, GPIO_11_F, GPIO_12_F, GPIO_13_F, GPIO_14_F, GPIO_15_F, GPIO_16_F, GPIO_1_F, GPIO_2_F, GPIO_3_F, GPIO_4_F, GPIO_5_F, GPIO_6_F, GPIO_7_F, GPIO_8_F, GPIO_9_F, PMOD1_1, PMOD1_2, PMOD1_3, PMOD1_4, PMOD1_5, PMOD1_6, PMOD1_7, PMOD1_8, PMOD2_1, PMOD2_2, PMOD2_3, PMOD2_4, PMOD2_5, PMOD2_6, PMOD2_7, PMOD2_8, ~CE~_RAM, ~OE~_RAM, ~WE~_RAM
- net labels removed: +1V8, CLK_F, GPIO_1, GPIO_10, GPIO_11, GPIO_12, GPIO_13, GPIO_14, GPIO_15, GPIO_16, GPIO_2, GPIO_3, GPIO_4, GPIO_5, GPIO_6, GPIO_7, GPIO_8, GPIO_9, IO1_CLK0, RX_A_F, SW_USER1, SW_USER2
- wire segments 168 -> 16
- no-connect marks 3 -> 4
Other:
- moved on the sheet: U12

Commit message: component placement
Parts:
- U4: symbol CPLD_Altera:5M1270ZT144C5N -> rc2014_max_v-rescue:5M1270ZT144C5N-CPLD_Altera
Changed lines of the file:
@@
 ~CE~_RAM
 $Comp
-L CPLD_Altera:5M1270ZT144C5N U4
+L rc2014_max_v-rescue:5M1270ZT144C5N-CPLD_Altera U4
 U 1 1 5D138C9B
 P 7850 720
+AR Path="/5D138C9B" Ref="U4"  Part="1"
+AR Path="/5CFABACD/5D138C9B" Ref="U4"  Part="1"
 F 0 "U4" H 8512 -357 50  0000 L CNN
 F 1 "5M1270ZT144C5N" H 8512 -448 50  0000 L CNN
@@
 $EndComp
 $Comp
-L CPLD_Altera:5M1270ZT144C5N U4
+L rc2014_max_v-rescue:5M1270ZT144C5N-CPLD_Altera U4
 U 2 1 5D1C9E99
 P 5240 3890
+AR Path="/5D1C9E99" Ref="U4"  Part="2"
+AR Path="/5CFABACD/5D1C9E99" Ref="U4"  Part="2"
 F 0 "U4" H 5902 2438 50  0000 L CNN
 F 1 "5M1270ZT144C5N" H 5902 2347 50  0000 L CNN
@@
 $EndComp
 $Comp
-L CPLD_Altera:5M1270ZT144C5N U4
+L rc2014_max_v-rescue:5M1270ZT144C5N-CPLD_Altera U4
 U 3 1 5D1FC2B4
 P 5210 670
+AR Path="/5D1FC2B4" Ref="U4"  Part="3"
+AR Path="/5CFABACD/5D1FC2B4" Ref="U4"  Part="3"
 F 0 "U4" H 5872 -622 50  0000 L CNN
 F 1 "5M1270ZT144C5N" H 5872 -713 50  0000 L CNN
@@
 $EndComp
 $Comp
-L CPLD_Altera:5M1270ZT144C5N U4
+L rc2014_max_v-rescue:5M1270ZT144C5N-CPLD_Altera U4
 U 4 1 5D22481B
 P 7880 3230
+AR Path="/5D22481B" Ref="U4"  Part="4"
+AR Path="/5CFABACD/5D22481B" Ref="U4"  Part="4"
 F 0 "U4" H 8648 1788 50  0000 L CNN
 F 1 "5M1270ZT144C5N" H 8648 1697 50  0000 L CNN
